File: SmartWatch V5/_autosave-SmartWatch V5.sch (KiCad schematic (older format))
At the start: 55 parts, among them J1 10118192-0001LF, J10 TestPad, J2 , J8 TestPad, J9 TestPad, Q1 FDN340P, Q2 MMBT3904, Q3 MMBT3904, Q4 FDN028N20, Q5 FDN028N20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

Commit message: Completed New Layout and Routing of Rev 5 (overall improved)
Connections:
- net BAT_ALRT: now also U6.31 (IO19); no longer U6.6 (IO34)
Changed lines of the file:
@@
 $EndDescr
-$Comp
-L RF_Module:ESP32-WROOM-32 U6
-U 1 1 5E6BFC95
-P 7350 2650
-F 0 "U6" H 6600 4250 50  0000 C CNN
-F 1 "ESP32-WROOM-32" H 6900 4150 50  0000 C CNN
-F 2 "RF_Module:ESP32-WROOM-32" H 7350 1150 50  0001 C CNN
-F 3 "https://www.espressif.com/sites/default/files/documentation/esp32-wroom-32_datasheet_en.pdf" H 7050 2700 50  0001 C CNN
-F 4 "1904-1010-1-ND" H 7350 2650 50  0001 C CNN "digikey"
-	1    7350 2650
-	1    0    0    -1
-$EndComp
 $Comp
 L power:+3.3V #PWR0101
@@
 Text Label 8350 3750 2    50   ~ 0
 CHG_STAT
-Text Label 8350 3650 2    50   ~ 0
-BAT_ALRT
-Wire Wire Line
-	7950 3650 8350 3650
+Wire Wire Line
+	7950 2750 8350 2750
 Wire Wire Line
 	7950 3750 8350 3750
@@
 NoConn ~ 4050 6800
 NoConn ~ 7950 1950
-NoConn ~ 7950 2750
 $Comp
 L Device:Thermistor TH1
@@
 Wire Wire Line
 	3550 1300 4050 1300
+$Comp
+L RF_Module:ESP32-WROOM-32 U6
+U 1 1 5E6BFC95
+P 7350 2650
+F 0 "U6" H 6600 4250 50  0000 C CNN
+F 1 "ESP32-WROOM-32" H 6900 4150 50  0000 C CNN
+F 2 "RF_Module:ESP32-WROOM-32" H 7350 1150 50  0001 C CNN
+F 3 "https://www.espressif.com/sites/default/files/documentation/esp32-wroom-32_datasheet_en.pdf" H 7050 2700 50  0001 C CNN
+F 4 "1904-1010-1-ND" H 7350 2650 50  0001 C CNN "digikey"
+	1    7350 2650
+	1    0    0    -1
+$EndComp
+Text Label 8350 2750 2    50   ~ 0
+BAT_ALRT
+NoConn ~ 7950 3650
 $EndSCHEMATC
